File: PCB/team build full layout.sch (EAGLE design)
At the start: 9 parts, among them IC1 ICL7663CPA, IC2 ICL7663CPA, IC3 ICL7663CPA

Commit message: Add files via upload
Parts:
- added CN1: 1X4-3.5MM, adafruit:1X4-3.5MM
- added DAMPER_POT: (no value), adafruit:PINHD-1X3CB
- added GPS: (no value), adafruit:PINHD-1X6-3.5MM
Connections:
- new net BL_GND: DAMPER_POT.2
- new net BR_VCC: DAMPER_POT.1
- new net CL: GPS.3
- new net DA: GPS.2
- new net RX: CN1.2
- new net RX_2: GPS.5
- new net TX: CN1.3
- new net TX_2: GPS.4
- new net VOLT_METER: DAMPER_POT.3
- net 3.3V: now also CN1.4
- net 5V: now also GPS.6
- net GND: now also CN1.1, GPS.1
