File: PCB/team build full layout.sch (EAGLE design)
At the start: 14 parts, among them CN1 1X4-3.5MM, IC1 ICL7663CPA, IC2 ICL7663CPA, IC3 ICL7663CPA

Commit message: first draft layout 07-08
Parts:
- removed BRAKE_OVER_TRAVEL_SWT: (no value), switch:255SB
- removed CN1: 1X4-3.5MM, adafruit:1X4-3.5MM
- removed DAMPER_POT: (no value), adafruit:PINHD-1X3CB
- added ACCELERATOR2, ACCELERATOR3, COOLANT_TEMP, WHEEL_SP1, WHEEL_SP2, WHEEL_SP3, WHEEL_SP4: (no value), adafruit:PINHD-1X3
- added ACCELEROMETER: 1X4-3.5MM, adafruit:1X4-3.5MM
- added BRAKE_SW: (no value), special:SW_DIP-1
- added CAN1_CLCH, U$10, U$6, U$7, U$8: CAN_BUS, F-E library custom components:CAN_BUS
- added CAN1_TEE, U$11, U$9: CAN_TEE, F-E library custom components:CAN_TEE
- added DAMPER_POT1, DAMPER_POT2, DAMPER_POT3, DAMPER_POT4: (no value), adafruit:PINHD-1X3CB
- added IC4: 7805T, adafruit:7805T
- added LED1, LED10, LED11, LED12, LED13, LED14, LED15, LED2, LED3, LED4, LED5, LED6, LED7, LED8, LED9: (no value), adafruit:LED3MM
- added MOTOR_CONTROLLER: 1X4-BIG, adafruit:1X4-BIG
- added R1, R10, R11, R12, R13, R14, R15, R16, R17, R3, R4, R5, R6, R7, R8, R9: 47k, rcl:R-US_0204/7
- added R2: 470k, rcl:R-US_0204/7
- U$1, U$2, U$3: value TEENSY40 -> TEENSY41; device teensy:TEENSY40 -> teensy:TEENSY41
- renumbered ROTARYENCODER to STEERING_ANGLE
Connections:
- removed net CL: GPS.3
- removed net DA: GPS.2
- removed net ON: BRAKE_OVER_TRAVEL_SWT.S
- removed net VOLT_METER: DAMPER_POT.3
- new net A1-L1: LED1.A, U$2.0-RX1/CS1/CRX2
- new net A1-L2: LED4.A, U$2.1-TX1/MISO1/CTX2
- new net A1-L3: LED7.A, U$2.2-OUT2
- new net A1-L4: LED10.A, U$2.3-LRCLK2
- new net A1-L5: LED13.A, U$2.4-BCLK2
- new net A2: DAMPER_POT1.3, U$1.16-A2/RX4/SCL1
- new net A2-L1: LED2.A, U$2.5-IN2
- new net A2-L2: LED5.A, U$2.6-OUT1D
- new net A2-L3: LED8.A, U$2.7-RX2/OUT1A
- new net A2-L4: LED11.A, U$2.8-TX2/IN1
- new net A2-L5: LED14.A, U$2.9-OUT1C
- new net A2_2: DAMPER_POT3.3, U$3.16-A2/RX4/SCL1
- new net A3: DAMPER_POT2.3, U$1.17-A3/TX4/SDA1
- new net A3-L1: LED3.A, U$2.10-CS/MQSR
- new net A3-L2: LED6.A, U$2.11-MOSI/CTX1
- new net A3-L3: LED9.A, U$2.12-MISO/MQSL
- new net A3-L4: LED12.A, U$2.24-A10/TX6/SCL2
- new net A3-L5: LED15.A, U$2.25-A11/RX6/SDA2
- new net A3_2: DAMPER_POT4.3, U$3.17-A3/TX4/SDA1
- new net ACC_DATA_OUT_1: ACCELERATOR3.2, R2.2, U$3.20-A6/TX5/LRCLK1
- new net ACC_DATA_OUT_2: ACCELERATOR2.2, R1.2, U$3.21-A7/RX5/BCLK1
- new net BR_SW: IC4.VO, U$3.24-A10/TX6/SCL2
- new net CRX_2: U$11.CRX, U$3.23-A9/CRX1/MCLK1
- new net CTX_2: U$11.CTX, U$3.22-A8/CTX1
- new net GND\: U$11.GND
- new net N$10: LED1.C, R3.2
- new net N$11: LED2.C, R4.2
- new net N$12: U$2.22-A8/CTX1, U$9.CTX
- new net N$13: U$2.23-A9/CRX1/MCLK1, U$9.CRX
- new net N$14: LED3.C, R5.2
- new net N$15: LED4.C, R6.2
- new net N$16: LED5.C, R7.2
- new net N$17: LED6.C, R8.2
- new net N$18: LED7.C, R9.2
- new net N$19: LED10.C, R10.2
- new net N$2: CAN1_TEE.CRX, U$1.23-A9/CRX1/MCLK1
- new net N$20: LED8.C, R11.2
- new net N$21: LED9.C, R12.2
- new net N$22: LED11.C, R13.2
- new net N$23: LED12.C, R14.2
- new net N$24: LED13.C, R15.2
- new net N$25: LED14.C, R16.2
- new net N$26: LED15.C, R17.2
- new net N$3: CAN1_TEE.CTX, U$1.22-A8/CTX1
- new net N$4: BRAKE_SW.1, IC4.VI
- new net N$6: U$2.17-A3/TX4/SDA1, U$4.SDA
- new net N$7: U$2.16-A2/RX4/SCL1, U$4.SCL
- new net N$8: U$2.18-A4/SDA0, U$5.SDA
- new net N$9: U$2.19-A5/SCL0, U$5.SCL
- new net SCL: GPS.3, U$1.24-A10/TX6/SCL2
- new net SDA: GPS.2, U$1.25-A11/RX6/SDA2
- new net WH_SP1_D: U$1.18-A4/SDA0, WHEEL_SP1.2
- new net WH_SP2_D: U$1.19-A5/SCL0, WHEEL_SP2.2
- new net WH_SP3_D: U$3.18-A4/SDA0, WHEEL_SP3.2
- new net WH_SP4_D: U$3.19-A5/SCL0, WHEEL_SP4.2
- net 12V: now also BRAKE_SW.2, WHEEL_SP1.1, WHEEL_SP2.1, WHEEL_SP3.1, WHEEL_SP4.1; no longer BRAKE_OVER_TRAVEL_SWT.P, STEERING_ANGLE.VCC
- net 3.3V: now also ACCELERATOR2.1, ACCELERATOR3.1, ACCELEROMETER.4, CAN1_TEE.3.3, U$11.3.3, U$4.VIO, U$5.VIO, U$9.3.3; no longer CN1.4
- net 5V: now also STEERING_ANGLE.VCC, U$4.VCC, U$5.VCC
- net BL_GND: now also DAMPER_POT3.2, DAMPER_POT4.2; no longer DAMPER_POT.2
- net BR_VCC: now also DAMPER_POT1.1, DAMPER_POT2.1, DAMPER_POT3.1, DAMPER_POT4.1; no longer DAMPER_POT.1
- net GND: now also ACCELERATOR2.3, ACCELERATOR3.3, ACCELEROMETER.1, CAN1_TEE.GND, COOLANT_TEMP.3, DAMPER_POT1.2, DAMPER_POT2.2, IC4.GND, R1.1, R10.1, R11.1, R12.1, R13.1, R14.1, R15.1, R16.1, R17.1, R2.1, R3.1, R4.1, R5.1, R6.1, R7.1, R8.1, R9.1, U$1.GND4, U$1.GND5, U$1.GND6, U$2.GND4, U$2.GND5, U$2.GND6, U$3.GND4, U$3.GND5, U$3.GND6, U$4.GND, U$5.GND, U$9.GND, WHEEL_SP1.3, WHEEL_SP2.3, WHEEL_SP3.3, WHEEL_SP4.3; no longer BRAKE_OVER_TRAVEL_SWT.O, CN1.1
- net RX: now also ACCELEROMETER.2, U$1.35/TX8; no longer CN1.2
- net RX_2: now also U$1.29-TX7
- net T2_DP_1: now also U$3.14-A0/TX3/SPDIF_OUT; no longer U$3.14-A0/TX3/S-PDIF_IN
- net TX: now also ACCELEROMETER.3, U$1.34-RX8; no longer CN1.3
- net TX_2: now also U$1.28-RX7
Other:
- note added: "LED dashboard display"
- note added: "Not sure how to use at the moment"
- note added: "edit at a later date. Only two pins"
- note added: "need to edit this voltage regulator as needed"
- moved on the sheet: GPS, IC2, IC3, U$4, U$5
