File: PCB/team dashboard display.sch (EAGLE design)
At the start: 36 parts, among them IC3 ICL7663CPA

Commit message: Stress board for Wheat bridge and edits
Created the Wheat bridge board with the different stress gauges in the F-E library. There were some minor edits that the other boards needed as well.
Connections:
- net 5V: now also U$2.VIN
Changed lines of the file:
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@@
 <label x="15.24" y="72.39" size="1.778" layer="95"/>
+</segment>
+<segment>
+<pinref part="U$2" gate="G$1" pin="VIN"/>
+<wire x1="91.44" y1="120.65" x2="91.44" y2="121.92" width="0.1524" layer="91"/>
+<label x="91.44" y="121.92" size="1.778" layer="95"/>
 </segment>
 </net>
