File: PCB/team back ECU.brd (EAGLE design)
At the start: 69.5 x 69.8 mm, 12 parts, among them IC2 ICL7663CPA

Commit message: Updated ECU and Strain Gauge board
Parts:
- removed CAN1_CLCH: CAN_BUS, F-E library custom components:CAN_BUS
- removed IC2: ICL7663CPA, maxim:DIL08
- added PWR_H: (no value), adafruit:1X03
- moved WHEEL_SP1 12.7 mm to (52.1, 59.7)
- moved WHEEL_SP2 12.7 mm to (52.1, 54.6)
- moved GPS 12.7 mm to (85.1, 29.2)
- moved MOTOR_CONTROLLER 12.7 mm to (69.8, 57.1)
- moved DAMPER_POT1 10.2 mm to (64.8, 57.1)
- moved DAMPER_POT2 10.2 mm to (61.0, 57.1)
- moved CAN1_TEE 3.81 mm to (45.7, 26.7)
- moved COOLANT_TEMP 3.59 mm to (63.5, 31.8)
Connections:
- net 12V: now also PWR_H.3; no longer IC2.8
- net 3.3V: now also U$1.3V3-1; no longer IC2.3
- net 5V: now also PWR_H.2, U$1.VIN; no longer IC2.2
- net GND: now also PWR_H.1; no longer IC2.4
Routing:
- net 5V: track 58.6 -> 92.2 mm
- net 12V: track 43.7 -> 14.8 mm
- net SCL: track 26.5 -> 13.8 mm
- net RX_2: track 19.6 -> 6.95 mm
- net WH_SP2_D: track 18.1 -> 5.39 mm
- net TX_2: track 19.2 -> 6.55 mm
- net SDA: track 19.5 -> 6.81 mm
- net WH_SP1_D: track 24.2 -> 12.4 mm
- net A_MC: track 22.7 -> 11.5 mm
- net A3: track 14.0 -> 3.81 mm
- net A2: track 14.5 -> 4.34 mm
- net N$3: track 24.0 -> 19.5 mm
- net N$2: track 25.9 -> 22.4 mm
- net 3.3V: track 75.9 -> 72.6 mm
Other:
- board size 69.5 x 69.8 mm -> 69.5 x 39.4 mm
